File: pcb/nestWidget.brd (EAGLE design)
At the start: 160 x 100 mm, 25 parts, among them K1 AQW27A, K2 AQY22SOP, U1 PIC16F1823ST

Commit message: First commit. -Most things there.
Parts:
- added K3: AQY22SOP, relay:SOP04
- K1: value AQW27A -> AQY22SOP; device relay:AQW27-SMD08 -> relay:SOP04
- moved K2 97.0 mm to (-41.9, -74.9)
- moved K1 74.1 mm to (-41.9, -66.0)
Connections:
- net N$2: now also K2.1; no longer K1.3
- net N$3: now also K3.1; no longer K2.1
- net N$4: now also K3.4; no longer K2.4
- net N$5: now also K2.4; no longer K1.6
- net N$6: now also K1.4; no longer K1.8
- net RELAY_FAN_OUT: now also K1.3; no longer K1.7
- net RELAY_HEATER: now also K2.2; no longer K1.4
- net RELAY_HEATER_OUT: now also K2.3; no longer K1.5
- net RELAY_MAINS: now also K3.2; no longer K2.2
- net RELAY_MAINS_OUT: now also K3.3; no longer K2.3
Changed lines of the file:
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@@
 <element name="JP2" library="pinhead" package="1X02" value="" x="-43.18" y="29.21"/>
 <element name="JP3" library="pinhead" package="1X06" value="" x="-25.4" y="29.21"/>
-<element name="K1" library="relay" package="AQW27-SMD08" value="AQW27A" x="-34.29" y="7.62"/>
-<element name="K2" library="relay" package="SOP04" value="AQY22SOP" x="-17.78" y="19.05">
+<element name="K3" library="relay" package="SOP04" value="AQY22SOP" x="-17.78" y="19.05">
 <attribute name="OC_FARNELL" value="unknown" x="-17.78" y="19.05" size="1.778" layer="27" display="off"/>
 <attribute name="OC_NEWARK" value="unknown" x="-17.78" y="19.05" size="1.778" layer="27" display="off"/>
@@
 <element name="JP8" library="pinhead" package="1X03" value="" x="-41.91" y="-52.07"/>
 <element name="JP7" library="pinhead" package="1X03" value="" x="-41.91" y="-58.42"/>
+<element name="K1" library="relay" package="SOP04" value="AQY22SOP" x="-41.91" y="-66.04">
+<attribute name="OC_FARNELL" value="unknown" x="-41.91" y="-66.04" size="1.778" layer="27" display="off"/>
+<attribute name="MF" value="" x="-41.91" y="-66.04" size="1.778" layer="27" display="off"/>
+<attribute name="MPN" value="" x="-41.91" y="-66.04" size="1.778" layer="27" display="off"/>
+<attribute name="OC_NEWARK" value="unknown" x="-41.91" y="-66.04" size="1.778" layer="27" display="off"/>
+</element>
+<element name="K2" library="relay" package="SOP04" value="AQY22SOP" x="-41.91" y="-74.93">
+<attribute name="OC_FARNELL" value="unknown" x="-41.91" y="-74.93" size="1.778" layer="27" display="off"/>
+<attribute name="MF" value="" x="-41.91" y="-74.93" size="1.778" layer="27" display="off"/>
+<attribute name="MPN" value="" x="-41.91" y="-74.93" size="1.778" layer="27" display="off"/>
+<attribute name="OC_NEWARK" value="unknown" x="-41.91" y="-74.93" size="1.778" layer="27" display="off"/>
+</element>
 </elements>
 <signals>
@@
 <contactref element="R1" pad="2"/>
 <contactref element="K1" pad="1"/>
-<wire x1="-41.91" y1="2.12" x2="-43.6" y2="-2.54" width="0" layer="19" extent="1-1"/>
+<wire x1="-43.6" y1="-2.54" x2="-43.18" y2="-69.04" width="0" layer="19" extent="1-1"/>
 </signal>
 <signal name="N$2">
 <contactref element="R2" pad="2"/>
-<contactref element="K1" pad="3"/>
-<wire x1="-31.75" y1="2.12" x2="-43.6" y2="-6.35" width="0" layer="19" extent="1-1"/>
+<contactref element="K2" pad="1"/>
+<wire x1="-43.6" y1="-6.35" x2="-43.18" y2="-77.93" width="0" layer="19" extent="1-1"/>
 </signal>
 <signal name="N$3">
 <contactref element="R3" pad="2"/>
-<contactref element="K2" pad="1"/>
+<contactref element="K3" pad="1"/>
 <wire x1="-19.05" y1="16.05" x2="-43.6" y2="-10.16" width="0" layer="19" extent="1-1"/>
 </signal>
 <signal name="N$4">
-<contactref element="K2" pad="4"/>
+<contactref element="K3" pad="4"/>
 <contactref element="R6" pad="1"/>
 <wire x1="-19.05" y1="22.05" x2="-45.3" y2="-21.59" width="0" layer="19" extent="1-1"/>
@@
 <signal name="N$5">
 <contactref element="R5" pad="1"/>
-<contactref element="K1" pad="6"/>
-<wire x1="-31.75" y1="13.12" x2="-45.3" y2="-17.78" width="0" layer="19" extent="1-1"/>
+<contactref element="K2" pad="4"/>
+<wire x1="-45.3" y1="-17.78" x2="-43.18" y2="-71.93" width="0" layer="19" extent="1-1"/>
 </signal>
 <signal name="N$6">
 <contactref element="R4" pad="1"/>
-<contactref element="K1" pad="8"/>
-<wire x1="-41.91" y1="13.12" x2="-45.3" y2="-13.97" width="0" layer="19" extent="1-1"/>
+<contactref element="K1" pad="4"/>
+<wire x1="-45.3" y1="-13.97" x2="-43.18" y2="-63.04" width="0" layer="19" extent="1-1"/>
 </signal>
 <signal name="RELAY_FAN">
+<contactref element="U1" pad="10"/>
 <contactref element="K1" pad="2"/>
-<contactref element="U1" pad="10"/>
-<wire x1="-17.13" y1="6.635" x2="-36.83" y2="2.12" width="0" layer="19" extent="1-1"/>
+<wire x1="-17.13" y1="6.635" x2="-40.64" y2="-69.04" width="0" layer="19" extent="1-1"/>
 </signal>
 <signal name="RELAY_HEATER">
-<contactref element="K1" pad="4"/>
 <contactref element="U1" pad="9"/>
-<wire x1="-16.48" y1="6.635" x2="-26.67" y2="2.12" width="0" layer="19" extent="1-1"/>
+<contactref element="K2" pad="2"/>
+<wire x1="-16.48" y1="6.635" x2="-40.64" y2="-77.93" width="0" layer="19" extent="1-1"/>
 </signal>
 <signal name="RELAY_MAINS">
-<contactref element="K2" pad="2"/>
+<contactref element="K3" pad="2"/>
 <contactref element="U1" pad="8"/>
 <wire x1="-16.51" y1="16.05" x2="-15.83" y2="6.635" width="0" layer="19" extent="1-1"/>
 </signal>
 <signal name="RELAY_FAN_OUT">
-<contactref element="K1" pad="7"/>
 <contactref element="JP4" pad="1"/>
-<wire x1="-36.83" y1="13.12" x2="-44.45" y2="-26.67" width="0" layer="19" extent="1-1"/>
+<contactref element="K1" pad="3"/>
+<wire x1="-44.45" y1="-26.67" x2="-40.64" y2="-63.04" width="0" layer="19" extent="1-1"/>
 </signal>
 <signal name="RELAY_HEATER_OUT">
-<contactref element="K1" pad="5"/>
 <contactref element="JP5" pad="1"/>
-<wire x1="-26.67" y1="13.12" x2="-44.45" y2="-33.02" width="0" layer="19" extent="1-1"/>
+<contactref element="K2" pad="3"/>
+<wire x1="-44.45" y1="-33.02" x2="-40.64" y2="-71.93" width="0" layer="19" extent="1-1"/>
 </signal>
 <signal name="RELAY_MAINS_OUT">
-<contactref element="K2" pad="3"/>
+<contactref element="K3" pad="3"/>
 <contactref element="JP6" pad="1"/>
 <wire x1="-16.51" y1="22.05" x2="-44.45" y2="-39.37" width="0" layer="19" extent="1-1"/>
