File: pcb/nestWidget.sch (EAGLE design)
At the start: 13 parts, among them T1 TICP206, U1 PIC16F1823ST

Commit message: Added most parts.
Parts:
- removed T1: TICP206, triac:TICP206
- added JP4, JP5, JP6: (no value), pinhead:PINHD-1X2
- added JP7, JP8: (no value), pinhead:PINHD-1X3
- added K1: AQW27A, relay:AQW27A
- added K2: AQY22SOP, relay:AQY22SOP
- added R1, R2, R3: 1.6K, rcl:R-US_R0603
- added R4, R5, R6: (no value), rcl:R-US_R0603
Connections:
- new net LED1: LED1.C, U1.RC3
- new net LED2: LED2.C, U1.RC4
- new net N$1: K1A.A, R1.2
- new net N$2: K1B.A, R2.2
- new net N$3: K2.A, R3.2
- new net N$4: K2.DS1, R6.1
- new net N$5: K1B.D1, R5.1
- new net N$6: K1A.D1, R4.1
- new net RELAY_FAN: K1A.K, U1.RC0
- new net RELAY_FAN_OUT: JP4.1, K1A.D2
- new net RELAY_HEATER: K1B.K, U1.RC1
- new net RELAY_HEATER_OUT: JP5.1, K1B.D2
- new net RELAY_MAINS: K2.K, U1.RC2
- new net RELAY_MAINS_OUT: JP6.1, K2.DS2
- new net V+: JP8.2, R4.2, R5.2, R6.2
- new net V-: JP4.2, JP5.2, JP6.2, JP7.2
- net +12V: now also JP8.3
- net +3V3: now also R1.1, R2.1, R3.1
- net 24V0_AC_L: now also JP8.1
- net 24V0_AC_N: now also JP7.1
- net GND: now also JP7.3
Other:
- note added: "3. MUST ONLY USE LOW-POWER OSC MODES IF USING LDO FROM 12V RAIL"
- moved on the sheet: LED1, LED2, R7, R8

Commit message: First commit. -Most things there.
Parts:
- added K3: AQY22SOP, relay:AQY22SOP
- K1: value AQW27A -> AQY22SOP; device relay:AQW27A -> relay:AQY22SOP
Connections:
- net N$1: now also K1.A; no longer K1A.A
- net N$2: now also K2.A; no longer K1B.A
- net N$3: now also K3.A; no longer K2.A
- net N$4: now also K3.DS1; no longer K2.DS1
- net N$5: now also K2.DS1; no longer K1B.D1
- net N$6: now also K1.DS1; no longer K1A.D1
- net RELAY_FAN: now also K1.K; no longer K1A.K
- net RELAY_FAN_OUT: now also K1.DS2; no longer K1A.D2
- net RELAY_HEATER: now also K2.K; no longer K1B.K
- net RELAY_HEATER_OUT: now also K2.DS2; no longer K1B.D2
- net RELAY_MAINS: now also K3.K; no longer K2.K
- net RELAY_MAINS_OUT: now also K3.DS2; no longer K2.DS2
Other:
- moved on the sheet: K2
Changed lines of the file:
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@@
 <part name="+3V3" library="supply1" deviceset="+3V3" device=""/>
 <part name="GND4" library="supply1" deviceset="GND" device=""/>
-<part name="K1" library="relay" deviceset="AQW27" device="A"/>
-<part name="K2" library="relay" deviceset="AQY*" device="SOP" technology="22"/>
+<part name="K3" library="relay" deviceset="AQY*" device="SOP" technology="22"/>
 <part name="R1" library="rcl" deviceset="R-US_" device="R0603" value="1.6K"/>
 <part name="R2" library="rcl" deviceset="R-US_" device="R0603" value="1.6K"/>
@@
 <part name="JP7" library="pinhead" deviceset="PINHD-1X3" device=""/>
 <part name="GND5" library="supply1" deviceset="GND" device=""/>
+<part name="K1" library="relay" deviceset="AQY*" device="SOP" technology="22"/>
+<part name="K2" library="relay" deviceset="AQY*" device="SOP" technology="22"/>
 </parts>
 <sheets>
@@
 <instance part="+3V3" gate="G$1" x="259.08" y="241.3"/>
 <instance part="GND4" gate="1" x="259.08" y="218.44"/>
-<instance part="K1" gate="A" x="299.72" y="142.24"/>
-<instance part="K1" gate="B" x="299.72" y="119.38"/>
-<instance part="K2" gate="G$1" x="299.72" y="96.52"/>
+<instance part="K3" gate="G$1" x="299.72" y="96.52"/>
 <instance part="R1" gate="G$1" x="274.32" y="144.78"/>
 <instance part="R2" gate="G$1" x="274.32" y="121.92"/>
@@
 <instance part="JP7" gate="A" x="297.18" y="162.56"/>
 <instance part="GND5" gate="1" x="271.78" y="154.94"/>
+<instance part="K1" gate="G$1" x="299.72" y="142.24"/>
+<instance part="K2" gate="G$1" x="299.72" y="119.38"/>
 </instances>
 <busses>
@@
 <segment>
 <pinref part="R1" gate="G$1" pin="2"/>
-<pinref part="K1" gate="A" pin="A"/>
 <wire x1="279.4" y1="144.78" x2="289.56" y2="144.78" width="0.1524" layer="91"/>
+<pinref part="K1" gate="G$1" pin="A"/>
 </segment>
 </net>
@@
 <segment>
 <pinref part="R2" gate="G$1" pin="2"/>
-<pinref part="K1" gate="B" pin="A"/>
 <wire x1="279.4" y1="121.92" x2="289.56" y2="121.92" width="0.1524" layer="91"/>
+<pinref part="K2" gate="G$1" pin="A"/>
 </segment>
 </net>
@@
 <segment>
 <pinref part="R3" gate="G$1" pin="2"/>
-<pinref part="K2" gate="G$1" pin="A"/>
+<pinref part="K3" gate="G$1" pin="A"/>
 <wire x1="279.4" y1="99.06" x2="289.56" y2="99.06" width="0.1524" layer="91"/>
 </segment>
@@
 <net name="N$4" class="0">
 <segment>
-<pinref part="K2" gate="G$1" pin="DS1"/>
+<pinref part="K3" gate="G$1" pin="DS1"/>
 <pinref part="R6" gate="G$1" pin="1"/>
 <wire x1="309.88" y1="99.06" x2="314.96" y2="99.06" width="0.1524" layer="91"/>
@@
 <segment>
 <pinref part="R5" gate="G$1" pin="1"/>
-<pinref part="K1" gate="B" pin="D1"/>
 <wire x1="314.96" y1="121.92" x2="309.88" y2="121.92" width="0.1524" layer="91"/>
+<pinref part="K2" gate="G$1" pin="DS1"/>
 </segment>
 </net>
@@
 <segment>
 <pinref part="R4" gate="G$1" pin="1"/>
-<pinref part="K1" gate="A" pin="D1"/>
 <wire x1="314.96" y1="144.78" x2="309.88" y2="144.78" width="0.1524" layer="91"/>
+<pinref part="K1" gate="G$1" pin="DS1"/>
 </segment>
 </net>
 <net name="RELAY_FAN" class="0">
 <segment>
-<pinref part="K1" gate="A" pin="K"/>
 <wire x1="289.56" y1="139.7" x2="266.7" y2="139.7" width="0.1524" layer="91"/>
 <label x="269.24" y="139.7" size="1.778" layer="95"/>
+<pinref part="K1" gate="G$1" pin="K"/>
 </segment>
 <segment>
@@
 <net name="RELAY_HEATER" class="0">
 <segment>
-<pinref part="K1" gate="B" pin="K"/>
 <wire x1="266.7" y1="116.84" x2="289.56" y2="116.84" width="0.1524" layer="91"/>
 <label x="269.24" y="116.84" size="1.778" layer="95"/>
+<pinref part="K2" gate="G$1" pin="K"/>
 </segment>
 <segment>
@@
 <net name="RELAY_MAINS" class="0">
 <segment>
-<pinref part="K2" gate="G$1" pin="K"/>
+<pinref part="K3" gate="G$1" pin="K"/>
 <wire x1="266.7" y1="93.98" x2="289.56" y2="93.98" width="0.1524" layer="91"/>
 <label x="269.24" y="93.98" size="1.778" layer="95"/>
@@
 <net name="RELAY_FAN_OUT" class="0">
 <segment>
-<pinref part="K1" gate="A" pin="D2"/>
 <wire x1="309.88" y1="139.7" x2="342.9" y2="139.7" width="0.1524" layer="91"/>
 <label x="312.42" y="139.7" size="1.778" layer="95"/>
 <pinref part="JP4" gate="G$1" pin="1"/>
+<pinref part="K1" gate="G$1" pin="DS2"/>
 </segment>
 </net>
 <net name="RELAY_HEATER_OUT" class="0">
 <segment>
-<pinref part="K1" gate="B" pin="D2"/>
 <wire x1="309.88" y1="116.84" x2="342.9" y2="116.84" width="0.1524" layer="91"/>
 <label x="312.42" y="116.84" size="1.778" layer="95"/>
 <pinref part="JP5" gate="G$1" pin="1"/>
+<pinref part="K2" gate="G$1" pin="DS2"/>
 </segment>
 </net>
 <net name="RELAY_MAINS_OUT" class="0">
 <segment>
-<pinref part="K2" gate="G$1" pin="DS2"/>
+<pinref part="K3" gate="G$1" pin="DS2"/>
 <wire x1="309.88" y1="93.98" x2="342.9" y2="93.98" width="0.1524" layer="91"/>
 <label x="312.42" y="93.98" size="1.778" layer="95"/>
